Commit message: senosrs added

File: body.urdf (robot description, URDF)
Before this commit: robot robot, 3 links, 2 joints
Joints:
- removed joint FL_Torso
- removed joint Torso_BL
- added joint Torso_BackLeg: type revolute, parent Torso, child BackLeg, origin xyz=2 0 1 rpy=0 0 0, axis 0 1 0, limit lower=-3.14159 upper=3.14159 effort=0.0 velocity=0.0
- added joint Torso_FrontLeg: type revolute, parent Torso, child FrontLeg, origin xyz=1 0 1 rpy=0 0 0, axis 0 1 0, limit lower=-3.14159 upper=3.14159 effort=0.0 velocity=0.0

Commit message: unbiased quadruped

File: body.urdf (robot description, URDF)
Before this commit: robot robot, 3 links, 2 joints
Links:
- added link BackLowerLeg, mass 1; collision box size=0.2 0.2 1; visual box size=0.2 0.2 1
- added link FrontLowerLeg, mass 1; collision box size=0.2 0.2 1; visual box size=0.2 0.2 1
- added link LeftLeg, mass 1; collision box size=1 0.2 0.2; visual box size=1 0.2 0.2
- added link LeftLowerLeg, mass 1; collision box size=0.2 0.2 1; visual box size=0.2 0.2 1
- added link RightLeg, mass 1; collision box size=1 0.2 0.2; visual box size=1 0.2 0.2
- added link RightLowerLeg, mass 1; collision box size=0.2 0.2 1; visual box size=0.2 0.2 1
- link BackLeg: geometry collision box size=0.2 1 0.2; visual box size=0.2 1 0.2
- link FrontLeg: geometry collision box size=0.2 1 0.2; visual box size=0.2 1 0.2
Joints:
- added joint BackLeg_BackLowerLeg: type revolute, parent BackLeg, child BackLowerLeg, origin xyz=0 1 0 rpy=0 0 0, axis 1 0 0, limit lower=-3.14159 upper=3.14159 effort=0.0 velocity=0.0
- added joint FrontLeg_FrontLowerLeg: type revolute, parent FrontLeg, child FrontLowerLeg, origin xyz=0 -1 0 rpy=0 0 0, axis 1 0 0, limit lower=-3.14159 upper=3.14159 effort=0.0 velocity=0.0
- added joint LeftLeg_LeftLowerLeg: type revolute, parent LeftLeg, child LeftLowerLeg, origin xyz=-1 0 0 rpy=0 0 0, axis 0 1 0, limit lower=-3.14159 upper=3.14159 effort=0.0 velocity=0.0
- added joint RightLeg_RightLowerLeg: type revolute, parent RightLeg, child RightLowerLeg, origin xyz=1 0 0 rpy=0 0 0, axis 0 1 0, limit lower=-3.14159 upper=3.14159 effort=0.0 velocity=0.0
- added joint Torso_LeftLeg: type revolute, parent Torso, child LeftLeg, origin xyz=-0.5 0 1 rpy=0 0 0, axis 0 1 0, limit lower=-3.14159 upper=3.14159 effort=0.0 velocity=0.0
- added joint Torso_RightLeg: type revolute, parent Torso, child RightLeg, origin xyz=0.5 0 1 rpy=0 0 0, axis 0 1 0, limit lower=-3.14159 upper=3.14159 effort=0.0 velocity=0.0
- joint Torso_BackLeg: axis 0 1 0 -> 1 0 0; origin xyz=2 0 1 rpy=0 0 0 -> xyz=0 0.5 1 rpy=0 0 0
- joint Torso_FrontLeg: axis 0 1 0 -> 1 0 0; origin xyz=1 0 1 rpy=0 0 0 -> xyz=0 -0.5 1 rpy=0 0 0

Commit message: dog moving towards ball

File: body.urdf (robot description, URDF)
Before this commit: robot robot, 9 links, 8 joints
Links:
- removed link BackLeg
- removed link BackLowerLeg
- removed link FrontLeg
- removed link FrontLowerLeg
- removed link LeftLeg
- removed link LeftLowerLeg
- removed link RightLeg
- removed link RightLowerLeg
- added link BackLeftLeg, mass 0.3; collision box size=0.2 0.2 0.5; visual box size=0.2 0.2 0.5
- added link BackLowerLeftLeg, mass 0.2; collision box size=0.2 0.2 0.5; visual box size=0.2 0.2 0.5
- added link BackLowerRightLeg, mass 0.2; collision box size=0.2 0.2 0.5; visual box size=0.2 0.2 0.5
- added link BackRightLeg, mass 0.3; collision box size=0.2 0.2 0.5; visual box size=0.2 0.2 0.5
- added link FrontLeftLeg, mass 0.3; collision box size=0.2 0.2 0.5; visual box size=0.2 0.2 0.5
- added link FrontLowerLeftLeg, mass 0.2; collision box size=0.2 0.2 0.5; visual box size=0.2 0.2 0.5
- added link FrontLowerRightLeg, mass 0.2; collision box size=0.2 0.2 0.5; visual box size=0.2 0.2 0.5
- added link FrontRightLeg, mass 0.3; collision box size=0.2 0.2 0.5; visual box size=0.2 0.2 0.5
- link Torso: geometry collision box size=1.5 0.5 0.5; visual box size=1.5 0.5 0.5
Joints:
- removed joint BackLeg_BackLowerLeg
- removed joint FrontLeg_FrontLowerLeg
- removed joint LeftLeg_LeftLowerLeg
- removed joint RightLeg_RightLowerLeg
- removed joint Torso_BackLeg
- removed joint Torso_FrontLeg
- removed joint Torso_LeftLeg
- removed joint Torso_RightLeg
- added joint BackLeftLeg_BackLowerLeftLeg: type revolute, parent BackLeftLeg, child BackLowerLeftLeg, origin xyz=0 0 -0.5 rpy=0 0 0, axis 0 1 0, limit lower=-3.14159 upper=3.14159 effort=0.0 velocity=0.0
- added joint BackRightLeg_BackLowerRightLeg: type revolute, parent BackRightLeg, child BackLowerRightLeg, origin xyz=0 0 -0.5 rpy=0 0 0, axis 0 1 0, limit lower=-3.14159 upper=3.14159 effort=0.0 velocity=0.0
- added joint FrontLeftLeg_FrontLowerLeftLeg: type revolute, parent FrontLeftLeg, child FrontLowerLeftLeg, origin xyz=0 0 -0.5 rpy=0 0 0, axis 0 1 0, limit lower=-3.14159 upper=3.14159 effort=0.0 velocity=0.0
- added joint FrontRightLeg_FrontLowerRightLeg: type revolute, parent FrontRightLeg, child FrontLowerRightLeg, origin xyz=0 0 -0.5 rpy=0 0 0, axis 0 1 0, limit lower=-3.14159 upper=3.14159 effort=0.0 velocity=0.0
- added joint Torso_BackLeftLeg: type revolute, parent Torso, child BackLeftLeg, origin xyz=0.75 -0.25 1 rpy=0 0 0, axis 0 1 0, limit lower=-3.14159 upper=3.14159 effort=0.0 velocity=0.0
- added joint Torso_BackRightLeg: type revolute, parent Torso, child BackRightLeg, origin xyz=0.75 0.25 1 rpy=0 0 0, axis 0 1 0, limit lower=-3.14159 upper=3.14159 effort=0.0 velocity=0.0
- added joint Torso_FrontLeftLeg: type revolute, parent Torso, child FrontLeftLeg, origin xyz=-0.75 -0.25 1 rpy=0 0 0, axis 0 1 0, limit lower=-3.14159 upper=3.14159 effort=0.0 velocity=0.0
- added joint Torso_FrontRightLeg: type revolute, parent Torso, child FrontRightLeg, origin xyz=-0.75 0.25 1 rpy=0 0 0, axis 0 1 0, limit lower=-3.14159 upper=3.14159 effort=0.0 velocity=0.0

Commit message: assignment 5 submission

File: body.urdf (robot description, URDF)
Before this commit: robot robot, 9 links, 8 joints
Links:
- link BackLowerLeftLeg: mass 0.2 -> 0.1; geometry collision box size=0.1 0.1 0.5; visual box size=0.1 0.1 0.5
- link BackLowerRightLeg: mass 0.2 -> 0.1; geometry collision box size=0.1 0.1 0.5; visual box size=0.1 0.1 0.5
- link FrontLowerLeftLeg: mass 0.2 -> 0.1; geometry collision box size=0.1 0.1 0.5; visual box size=0.1 0.1 0.5
- link FrontLowerRightLeg: mass 0.2 -> 0.1; geometry collision box size=0.1 0.1 0.5; visual box size=0.1 0.1 0.5

Commit message: basic snake

File: body.urdf (robot description, URDF)
Before this commit: robot robot, 9 links, 8 joints
Links:
- removed link BackLeftLeg
- removed link BackLowerLeftLeg
- removed link BackLowerRightLeg
- removed link BackRightLeg
- removed link FrontLeftLeg
- removed link FrontLowerLeftLeg
- removed link FrontLowerRightLeg
- removed link FrontRightLeg
- removed link Torso
- added link 0, mass 1; collision box size=1 1 1; visual box size=1 1 1
- added link 1, mass 1; collision box size=1 2.2285145312725243 1.8106573654122575; visual box size=1 2.2285145312725243 1.8106573654122575
- added link 2, mass 1; collision box size=2.5795599691928164 2.627646200381997 1; visual box size=2.5795599691928164 2.627646200381997 1
- added link 3, mass 1; collision box size=1.4048824678463987 1.526161849088667 1.8086883057488037; visual box size=1.4048824678463987 1.526161849088667 1.8086883057488037
Joints:
- removed joint BackLeftLeg_BackLowerLeftLeg
- removed joint BackRightLeg_BackLowerRightLeg
- removed joint FrontLeftLeg_FrontLowerLeftLeg
- removed joint FrontRightLeg_FrontLowerRightLeg
- removed joint Torso_BackLeftLeg
- removed joint Torso_BackRightLeg
- removed joint Torso_FrontLeftLeg
- removed joint Torso_FrontRightLeg
- added joint 0_1: type revolute, parent 0, child 1, origin xyz=-0.5 0 0.5 rpy=0 0 0, axis 0 1 0, limit lower=-3.14159 upper=3.14159 effort=0.0 velocity=0.0
- added joint 1_2: type revolute, parent 1, child 2, origin xyz=-1 0 0 rpy=0 0 0, axis 0 1 0, limit lower=-3.14159 upper=3.14159 effort=0.0 velocity=0.0
- added joint 2_3: type revolute, parent 2, child 3, origin xyz=-2.5795599691928164 0 0 rpy=0 0 0, axis 0 1 0, limit lower=-3.14159 upper=3.14159 effort=0.0 velocity=0.0

Commit message: snake with random sensors

File: body.urdf (robot description, URDF)
Before this commit: robot robot, 4 links, 3 joints
Links:
- added link 4, mass 0.008182334508450231; collision box size=0.1559659866071687 0.21687255133037775 0.24190383018507622; visual box size=0.1559659866071687 0.21687255133037775 0.24190383018507622
- added link 5, mass 0.02565017897110692; collision box size=0.47552012721984327 0.22504608659095526 0.23969006353758793; visual box size=0.47552012721984327 0.22504608659095526 0.23969006353758793
- added link 6, mass 0.004380931842327791; collision box size=0.1 0.4960074192404221 0.08832391759455294; visual box size=0.1 0.4960074192404221 0.08832391759455294
- added link 7, mass 0.01616710335193102; collision box size=0.3229612576688684 0.2069374257200875 0.24190383018507622; visual box size=0.3229612576688684 0.2069374257200875 0.24190383018507622
- link 0: mass 1 -> 0.002419038301850763; geometry collision box size=0.1 0.1 0.24190383018507622; visual box size=0.1 0.1 0.24190383018507622
- link 1: mass 1 -> 0.0035479292282532444; geometry collision box size=0.10385729771467234 0.21732509132161126 0.15719113834563692; visual box size=0.10385729771467234 0.21732509132161126 0.15719113834563692
- link 2: mass 1 -> 0.00305754476619518; geometry collision box size=0.34395439938850103 0.41850912007422664 0.02124061216360118; visual box size=0.34395439938850103 0.41850912007422664 0.02124061216360118
- link 3: mass 1 -> 0.018451281141038833; geometry collision box size=0.2880721754533712 0.26477834853863336 0.24190383018507622; visual box size=0.2880721754533712 0.26477834853863336 0.24190383018507622
Joints:
- added joint 3_4: type revolute, parent 3, child 4, origin xyz=-0.2880721754533712 0 0 rpy=0 0 0, axis 0 1 0, limit lower=-3.14159 upper=3.14159 effort=0.0 velocity=0.0
- added joint 4_5: type revolute, parent 4, child 5, origin xyz=-0.1559659866071687 0 0 rpy=0 0 0, axis 0 1 0, limit lower=-3.14159 upper=3.14159 effort=0.0 velocity=0.0
- added joint 5_6: type revolute, parent 5, child 6, origin xyz=-0.47552012721984327 0 0 rpy=0 0 0, axis 0 1 0, limit lower=-3.14159 upper=3.14159 effort=0.0 velocity=0.0
- added joint 6_7: type revolute, parent 6, child 7, origin xyz=-0.1 0 0 rpy=0 0 0, axis 0 1 0, limit lower=-3.14159 upper=3.14159 effort=0.0 velocity=0.0
- joint 0_1: origin xyz=-0.5 0 0.5 rpy=0 0 0 -> xyz=-0.05 0 0.12095191509253811 rpy=0 0 0
- joint 1_2: origin xyz=-1 0 0 rpy=0 0 0 -> xyz=-0.10385729771467234 0 0 rpy=0 0 0
- joint 2_3: origin xyz=-2.5795599691928164 0 0 rpy=0 0 0 -> xyz=-0.34395439938850103 0 0 rpy=0 0 0

Commit message: random morphology snake with colored links

File: body.urdf (robot description, URDF)
Before this commit: robot robot, 8 links, 7 joints
Links:
- added link 8, mass 1; collision box size=0.3 0.4056921349787851 0.9155577047240357; visual box size=0.3 0.4056921349787851 0.9155577047240357
- added link 9, mass 1; collision box size=0.3 0.4971409698400958 0.3; visual box size=0.3 0.4971409698400958 0.3
- link 0: mass 0.002419038301850763 -> 1; geometry collision box size=0.5690498264693129 0.5683868936101197 0.7105660191963005; visual box size=0.5690498264693129 0.5683868936101197 0.7105660191963005
- link 1: mass 0.0035479292282532444 -> 1; geometry collision box size=0.4975761725856461 0.3 0.3; visual box size=0.4975761725856461 0.3 0.3
- link 2: mass 0.00305754476619518 -> 1; geometry collision box size=0.4162634720114482 0.3 0.7926744384343946; visual box size=0.4162634720114482 0.3 0.7926744384343946
- link 3: mass 0.018451281141038833 -> 1; geometry collision box size=0.5120763917297637 0.6592399722951802 0.3; visual box size=0.5120763917297637 0.6592399722951802 0.3
- link 4: mass 0.008182334508450231 -> 1; geometry collision box size=0.40563446408540504 0.71257307447707 0.572830631275218; visual box size=0.40563446408540504 0.71257307447707 0.572830631275218
- link 5: mass 0.02565017897110692 -> 1; geometry collision box size=0.74629959689493 0.3 0.8778102480167495; visual box size=0.74629959689493 0.3 0.8778102480167495
- link 6: mass 0.004380931842327791 -> 1; geometry collision box size=0.6817888017073237 0.7590319147912976 0.3; visual box size=0.6817888017073237 0.7590319147912976 0.3
- link 7: mass 0.01616710335193102 -> 1; geometry collision box size=0.4226427512918066 0.5563863810826286 0.8948018888337373; visual box size=0.4226427512918066 0.5563863810826286 0.8948018888337373
Joints:
- added joint 7_8: type revolute, parent 7, child 8, origin xyz=-0.4226427512918066 0 0 rpy=0 0 0, axis 0 1 0, limit lower=-3.14159 upper=3.14159 effort=0.0 velocity=0.0
- added joint 8_9: type revolute, parent 8, child 9, origin xyz=-0.3 0 0 rpy=0 0 0, axis 0 1 0, limit lower=-3.14159 upper=3.14159 effort=0.0 velocity=0.0
- joint 0_1: origin xyz=-0.05 0 0.12095191509253811 rpy=0 0 0 -> xyz=-0.28452491323465645 0 0.5 rpy=0 0 0
- joint 1_2: origin xyz=-0.10385729771467234 0 0 rpy=0 0 0 -> xyz=-0.4975761725856461 0 0 rpy=0 0 0
- joint 2_3: origin xyz=-0.34395439938850103 0 0 rpy=0 0 0 -> xyz=-0.4162634720114482 0 0 rpy=0 0 0
- joint 3_4: origin xyz=-0.2880721754533712 0 0 rpy=0 0 0 -> xyz=-0.5120763917297637 0 0 rpy=0 0 0
- joint 4_5: origin xyz=-0.1559659866071687 0 0 rpy=0 0 0 -> xyz=-0.40563446408540504 0 0 rpy=0 0 0
- joint 5_6: origin xyz=-0.47552012721984327 0 0 rpy=0 0 0 -> xyz=-0.74629959689493 0 0 rpy=0 0 0
- joint 6_7: origin xyz=-0.1 0 0 rpy=0 0 0 -> xyz=-0.6817888017073237 0 0 rpy=0 0 0

Commit message: assignment 6 final submission

File: body.urdf (robot description, URDF)
Before this commit: robot robot, 10 links, 9 joints
Links:
- link 0: mass 1 -> 0.2804297768758938; geometry collision box size=0.9861102302435957 0.5687594921444434 0.5; visual box size=0.9861102302435957 0.5687594921444434 0.5
- link 1: mass 1 -> 0.2765398091829991; geometry collision box size=0.6763550305124796 0.8177356468346592 0.5; visual box size=0.6763550305124796 0.8177356468346592 0.5
- link 2: mass 1 -> 0.2774544189270528; geometry collision box size=0.7564143604308464 0.7336043138287787 0.5; visual box size=0.7564143604308464 0.7336043138287787 0.5
- link 3: mass 1 -> 0.3654554231966683; geometry collision box size=0.5 0.8676198679527402 0.8424321219360894; visual box size=0.5 0.8676198679527402 0.8424321219360894
- link 4: mass 1 -> 0.6009139294441457; geometry collision box size=0.921073523290417 0.8682577880158933 0.7513967032982304; visual box size=0.921073523290417 0.8682577880158933 0.7513967032982304
- link 5: mass 1 -> 0.23651459783539994; geometry collision box size=0.7294073663543429 0.6485116787825315 0.5; visual box size=0.7294073663543429 0.6485116787825315 0.5
- link 6: mass 1 -> 0.30775434736297347; geometry collision box size=0.5 0.7942231752985267 0.7749820376301587; visual box size=0.5 0.7942231752985267 0.7749820376301587
- link 7: mass 1 -> 0.32294480384295404; geometry collision box size=0.6948064473734541 0.9295964511088459 0.5; visual box size=0.6948064473734541 0.9295964511088459 0.5
- link 8: mass 1 -> 0.2555266954687705; geometry collision box size=0.7600958164766988 0.5698299085517651 0.5899601755191537; visual box size=0.7600958164766988 0.5698299085517651 0.5899601755191537
- link 9: mass 1 -> 0.125; geometry collision box size=0.5 0.5 0.5; visual box size=0.5 0.5 0.5
Joints:
- joint 0_1: origin xyz=-0.28452491323465645 0 0.5 rpy=0 0 0 -> xyz=-0.49305511512179784 0 0.5 rpy=0 0 0
- joint 1_2: origin xyz=-0.4975761725856461 0 0 rpy=0 0 0 -> xyz=-0.6763550305124796 0 0 rpy=0 0 0
- joint 2_3: origin xyz=-0.4162634720114482 0 0 rpy=0 0 0 -> xyz=-0.7564143604308464 0 0 rpy=0 0 0
- joint 3_4: origin xyz=-0.5120763917297637 0 0 rpy=0 0 0 -> xyz=-0.5 0 0 rpy=0 0 0
- joint 4_5: origin xyz=-0.40563446408540504 0 0 rpy=0 0 0 -> xyz=-0.921073523290417 0 0 rpy=0 0 0
- joint 5_6: origin xyz=-0.74629959689493 0 0 rpy=0 0 0 -> xyz=-0.7294073663543429 0 0 rpy=0 0 0
- joint 6_7: origin xyz=-0.6817888017073237 0 0 rpy=0 0 0 -> xyz=-0.5 0 0 rpy=0 0 0
- joint 7_8: origin xyz=-0.4226427512918066 0 0 rpy=0 0 0 -> xyz=-0.6948064473734541 0 0 rpy=0 0 0
- joint 8_9: origin xyz=-0.3 0 0 rpy=0 0 0 -> xyz=-0.7600958164766988 0 0 rpy=0 0 0

Commit message: assignment 7 done

File: body.urdf (robot description, URDF)
Before this commit: robot robot, 10 links, 9 joints
Links:
- removed link 5
- removed link 6
- removed link 7
- removed link 8
- removed link 9
- link 0: mass 0.2804297768758938 -> 1.0; geometry collision box size=0.810334856816814 0.4846484494599231 0.9074735004625607; visual box size=0.810334856816814 0.4846484494599231 0.9074735004625607
- link 1: mass 0.2765398091829991 -> 1.0; geometry collision box size=0.3 0.3 0.3; visual box size=0.3 0.3 0.3
- link 2: mass 0.2774544189270528 -> 1.0; geometry collision box size=0.3 0.639650065687351 0.3; visual box size=0.3 0.639650065687351 0.3
- link 3: mass 0.3654554231966683 -> 1.0; geometry collision box size=0.3 0.3 0.7625642966572603; visual box size=0.3 0.3 0.7625642966572603
- link 4: mass 0.6009139294441457 -> 1.0; geometry collision box size=0.3 0.3 0.7624542301729543; visual box size=0.3 0.3 0.7624542301729543
Joints:
- removed joint 3_4
- removed joint 4_5
- removed joint 5_6
- removed joint 6_7
- removed joint 7_8
- removed joint 8_9
- added joint 1_4: type revolute, parent 1, child 4, origin xyz=0.3 0.14096024700151158 -0.007323548943266389 rpy=0 0 0, axis 0 1 0, limit lower=-3.14159 upper=3.14159 effort=0.0 velocity=0.0
- joint 0_1: axis 0 1 0 -> 1 0 0; origin xyz=-0.49305511512179784 0 0.5 rpy=0 0 0 -> xyz=0.405167428408407 -0.15085294120795917 1.6662730065245803 rpy=0 0 0
- joint 1_2: axis 0 1 0 -> 1 0 0; origin xyz=-0.6763550305124796 0 0 rpy=0 0 0 -> xyz=0.0 0.040675570963032 0.12575038801910288 rpy=0 0 0
- joint 2_3: axis 0 1 0 -> 1 0 0; origin xyz=-0.7564143604308464 0 0 rpy=0 0 0 -> xyz=0.0 -0.1702984888414911 0.1123583483378499 rpy=0 0 0

Commit message: assignment 7 final submission

File: body.urdf (robot description, URDF)
Before this commit: robot robot, 5 links, 4 joints
Links:
- removed link 4
- link 0: geometry collision box size=0.7282253082507226 0.35969244080054563 0.42946969756653725; visual box size=0.7282253082507226 0.35969244080054563 0.42946969756653725
- link 1: geometry collision box size=0.8379878830772031 0.6703820369166472 0.5868278517792381; visual box size=0.8379878830772031 0.6703820369166472 0.5868278517792381
- link 2: geometry collision box size=0.4423523307006285 0.3 0.9087063630478518; visual box size=0.4423523307006285 0.3 0.9087063630478518
- link 3: geometry collision box size=0.36365826772003884 0.49983522051393836 0.377134366736421; visual box size=0.36365826772003884 0.49983522051393836 0.377134366736421
Joints:
- removed joint 1_4
- joint 0_1: axis 1 0 0 -> 0 0 1; origin xyz=0.405167428408407 -0.15085294120795917 1.6662730065245803 rpy=0 0 0 -> xyz=-0.3641126541253613 -0.15561715561268694 1.5054600812994774 rpy=0 0 0
- joint 1_2: origin xyz=0.0 0.040675570963032 0.12575038801910288 rpy=0 0 0 -> xyz=-0.12613526731399521 -0.10419280607872708 -0.29341392588961906 rpy=0 0 0
- joint 2_3: axis 1 0 0 -> 0 1 0; origin xyz=0.0 -0.1702984888414911 0.1123583483378499 rpy=0 0 0 -> xyz=0.07626593962324672 -0.12329584901494635 0.0 rpy=0 0 0

Commit message: more links more simulations

File: body.urdf (robot description, URDF)
Before this commit: robot robot, 4 links, 3 joints
Links:
- added link 4, mass 1.0; collision box size=0.3596493067212906 0.5590126010823101 0.8531597270192268; visual box size=0.3596493067212906 0.5590126010823101 0.8531597270192268
- link 0: geometry collision box size=0.5498211298945154 0.5989438370522632 0.30521666681945286; visual box size=0.5498211298945154 0.5989438370522632 0.30521666681945286
- link 1: geometry collision box size=0.8691797676202648 0.31812066723031796 0.3; visual box size=0.8691797676202648 0.31812066723031796 0.3
- link 2: geometry collision box size=0.3 0.5001924222331282 0.8858403356053971; visual box size=0.3 0.5001924222331282 0.8858403356053971
- link 3: geometry collision box size=0.3 0.5202622522507224 0.3; visual box size=0.3 0.5202622522507224 0.3
Joints:
- removed joint 2_3
- added joint 1_3: type revolute, parent 1, child 3, origin xyz=0.0 0.01076952651843585 0.13744403329013355 rpy=0 0 0, axis 1 0 0, limit lower=-3.14159 upper=3.14159 effort=0.0 velocity=0.0
- added joint 3_4: type revolute, parent 3, child 4, origin xyz=-0.25695284129478646 0.010630139340360662 0.15 rpy=0 0 0, axis 1 0 0, limit lower=-3.14159 upper=3.14159 effort=0.0 velocity=0.0
- joint 0_1: axis 0 0 1 -> 0 1 0; origin xyz=-0.3641126541253613 -0.15561715561268694 1.5054600812994774 rpy=0 0 0 -> xyz=0.2749105649472577 0.0008276146814578266 1.314605753781249 rpy=0 0 0
- joint 1_2: axis 1 0 0 -> 0 0 1; origin xyz=-0.12613526731399521 -0.10419280607872708 -0.29341392588961906 rpy=0 0 0 -> xyz=0.5017868060642755 0.15906033361515898 -0.10462594027696775 rpy=0 0 0
